Commit message: Some little updates

File: kuka_kr10_support/urdf/kr10r1100sixx_macro.xacro (robot description, xacro)
@@ -153,22 +153,32 @@
       <limit effort="0" lower="${radians(-350)}" upper="${radians(350)}" velocity="${radians(492)}"/>
     </joint>
-    <joint name="${prefix}joint_a6-flange" type="fixed">
+    <!-- <joint name="${prefix}joint_a6-flange" type="fixed">
       <parent link="${prefix}link_6"/>
       <child link="${prefix}flange"/>
       <origin xyz="0 0 0" rpy="0 0 0"/>
-    </joint>
+    </joint> -->
     <!-- ROS base_link to KUKA $ROBROOT coordinate system transform -->
-    <link name="${prefix}base" />
+    <!-- <link name="${prefix}base" />
     <joint name="${prefix}base_link-base" type="fixed">
       <origin xyz="0 0 0" rpy="0 0 0"/>
       <parent link="${prefix}base_link"/>
       <child link="${prefix}base"/>
-    </joint>
+    </joint> -->
     <!-- This frame corresponds to the $TOOL coordinate system in KUKA KRC controllers -->
     <link name="${prefix}tool0" />
-    <joint name="${prefix}flange-tool0" type="fixed">
+    <!-- <joint name="${prefix}flange-tool0" type="fixed">
       <parent link="${prefix}flange"/>
       <child link="${prefix}tool0"/>
       <origin xyz="0 0 0" rpy="0 ${radians(90)} 0"/>
+    </joint> -->
+    <joint name="${prefix}link_6-tool0" type="fixed">
+      <origin xyz="0.0 0 0" rpy="0 1.57079632679 0"/>
+      <parent link="${prefix}link_6"/>
+      <child link="${prefix}tool0"/>
+    </joint>
+    <joint name="${prefix}link_6-flange" type="fixed">
+      <origin xyz="0.0 0 0" rpy="0 1.57079632679 0"/>
+      <parent link="${prefix}link_6"/>
+      <child link="${prefix}flange"/>
     </joint>
   </xacro:macro>
