Commit message: Correct the velocity limits of joints

File: kuka_kr10_support/urdf/kr10r1100sixx_2_macro.xacro (robot description, xacro)
@@ -159,5 +159,5 @@
       <child link="${prefix}link_3"/>
       <axis xyz="0 1 0"/>
-      <limit effort="0" lower="${radians(-120)}" upper="${radians(156)}" velocity="${radians(225)}"/>
+      <limit effort="0" lower="${radians(-120)}" upper="${radians(156)}" velocity="${radians(330)}"/>
     </joint>
     <joint name="${prefix}joint_a4" type="revolute">
@@ -166,5 +166,5 @@
       <child link="${prefix}link_4"/>
       <axis xyz="-1 0 0"/>
-      <limit effort="0" lower="${radians(-185)}" upper="${radians(185)}" velocity="${radians(381)}"/>
+      <limit effort="0" lower="${radians(-185)}" upper="${radians(185)}" velocity="${radians(360)}"/>
     </joint>
     <joint name="${prefix}joint_a5" type="revolute">
@@ -173,5 +173,5 @@
       <child link="${prefix}link_5"/>
       <axis xyz="0 1 0"/>
-      <limit effort="0" lower="${radians(-120)}" upper="${radians(120)}" velocity="${radians(311)}"/>
+      <limit effort="0" lower="${radians(-120)}" upper="${radians(120)}" velocity="${radians(360)}"/>
     </joint>
     <joint name="${prefix}joint_a6" type="revolute">
@@ -180,5 +180,5 @@
       <child link="${prefix}link_6"/>
       <axis xyz="-11 0 0"/>
-      <limit effort="0" lower="${radians(-350)}" upper="${radians(350)}" velocity="${radians(492)}"/>
+      <limit effort="0" lower="${radians(-350)}" upper="${radians(350)}" velocity="${radians(433)}"/>
     </joint>
     <joint name="${prefix}link_6-tool0" type="fixed">

Commit message: Fix KR10 kinematics discrepancies

File: kuka_kr10_support/urdf/kr10r1100sixx_2_macro.xacro (robot description, xacro)
@@ -162,5 +162,5 @@
     </joint>
     <joint name="${prefix}joint_a4" type="revolute">
-      <origin xyz="0.205 0.0045 0.025" rpy="0 0 0"/>
+      <origin xyz="0.205 0.0 0.025" rpy="0 0 0"/>
       <parent link="${prefix}link_3"/>
       <child link="${prefix}link_4"/>
@@ -176,5 +176,5 @@
     </joint>
     <joint name="${prefix}joint_a6" type="revolute">
-      <origin xyz="0.067 0.00325 0" rpy="0 0 0"/>
+      <origin xyz="0.067 0 0" rpy="0 0 0"/>
       <parent link="${prefix}link_5"/>
       <child link="${prefix}link_6"/>

Commit message: Add isContinuous parameter for A6 so that it can be set up as a continuous joint

File: kuka_kr10_support/urdf/kr10r1100sixx_2_macro.xacro (robot description, xacro)
@@ -3,5 +3,6 @@
   <xacro:include filename="$(find kuka_resources)/urdf/common_constants.xacro"/>
   <xacro:include filename="$(find kuka_resources)/urdf/common_materials.xacro"/>
-  <xacro:macro name="kuka_kr10r1100sixx_2" params="prefix">
+  <xacro:property name="isContinuous" value="false"/>
+  <xacro:macro name="kuka_kr10r1100sixx_2" params="prefix isContinuous">
     <!-- links -->
     <link name="${prefix}base_link">
@@ -175,5 +176,5 @@
       <limit effort="0" lower="${radians(-120)}" upper="${radians(120)}" velocity="${radians(360)}"/>
     </joint>
-    <joint name="${prefix}joint_a6" type="revolute">
+    <!-- <joint name="${prefix}joint_a6" type="revolute">
       <origin xyz="0.067 0 0" rpy="0 0 0"/>
       <parent link="${prefix}link_5"/>
@@ -181,5 +182,22 @@
       <axis xyz="-11 0 0"/>
       <limit effort="0" lower="${radians(-350)}" upper="${radians(350)}" velocity="${radians(433)}"/>
-    </joint>
+    </joint> -->
+    <xacro:if value="${isContinuous == 'true'}">
+      <joint name="${prefix}joint_a6" type="continuous">
+        <origin xyz="0.067 0 0" rpy="0 0 0"/>
+        <parent link="${prefix}link_5"/>
+        <child link="${prefix}link_6"/>
+        <axis xyz="-11 0 0"/>
+      </joint>
+    </xacro:if>
+    <xacro:unless value="${isContinuous == 'true'}">
+      <joint name="${prefix}joint_a6" type="revolute">
+        <origin xyz="0.067 0 0" rpy="0 0 0"/>
+        <parent link="${prefix}link_5"/>
+        <child link="${prefix}link_6"/>
+        <axis xyz="-11 0 0"/>
+        <limit effort="0" lower="${radians(-350)}" upper="${radians(350)}" velocity="${radians(433)}"/>
+      </joint>
+    </xacro:unless>
     <joint name="${prefix}link_6-tool0" type="fixed">
       <origin xyz="0.023 0 0" rpy="0 1.57079632679 0"/>

Commit message: Add xyz and rpy parameters to that robroot can be transformed to match real kuka world

File: kuka_kr10_support/urdf/kr10r1100sixx_2_macro.xacro (robot description, xacro)
@@ -4,5 +4,5 @@
   <xacro:include filename="$(find kuka_resources)/urdf/common_materials.xacro"/>
   <xacro:property name="isContinuous" value="false"/>
-  <xacro:macro name="kuka_kr10r1100sixx_2" params="prefix isContinuous">
+  <xacro:macro name="kuka_kr10r1100sixx_2" params="prefix isContinuous base_xyz:='0 0 0' base_rpy:='0 0 0'">
     <!-- links -->
     <link name="${prefix}base_link">
@@ -211,10 +211,10 @@
     </joint>
     <!-- ROS base_link to KUKA $ROBROOT coordinate system transform -->
-    <!-- <link name="${prefix}base" />
+    <link name="${prefix}base" />
     <joint name="${prefix}base_link-base" type="fixed">
-      <origin xyz="0 0 0" rpy="0 0 0"/>
+      <origin xyz="${base_xyz}" rpy="${base_rpy}"/>
       <parent link="${prefix}base_link"/>
       <child link="${prefix}base"/>
-    </joint> -->
+    </joint>
     <!-- This frame corresponds to the $TOOL coordinate system in KUKA KRC controllers -->
     <!-- <link name="${prefix}tool0" />
