Commit message: Update KR16 R2010 URDF with KUKA-provided package

File: kuka_kr16_support/urdf/kr16r2010_2.xacro (robot description, xacro)
@@ -1,6 +1,8 @@
-<?xml version="1.0"?>
-<!--Generates a urdf from the macro in kr16_2_macro.xacro -->
-<robot name="kuka_kr16r2010_2" xmlns:xacro="http://wiki.ros.org/xacro">
-  <xacro:include filename="$(find kuka_kr16_support)/urdf/kr16r2010_2_macro.xacro" />
-  <xacro:kuka_kr16r2010_2 prefix=""/>
-</robot>
+<?xml version='1.0' encoding='utf-8'?>
+<robot name="kuka_kr16r2010_2" xmlns:xacro="http://www.ros.org/wiki/xacro">
+    <VERSION value="1.0.0" />
+    <!-- <xacro:arg default="r1_" name="prefix" /> -->
+    <xacro:arg default="" name="prefix" />
+    <xacro:include filename="$(find kuka_kr16_support)/urdf/kr16r2010_2/kr16r2010_2_macro.xacro" />
+    <xacro:kuka_kr16r2010_2 prefix="$(arg prefix)" />
+  </robot>

File: kuka_kr16_support/urdf/kr16r2010_2_macro.xacro (robot description, xacro)
@@ -1,229 +1,247 @@
-<?xml version="1.0"?>
-<robot xmlns:xacro="http://wiki.ros.org/xacro">
-  <xacro:include filename="$(find kuka_resources)/urdf/common_constants.xacro"/>
-  <xacro:include filename="$(find kuka_resources)/urdf/common_materials.xacro"/>
-  <xacro:macro name="kuka_kr16r2010_2" params="prefix">
-    <!-- LINKS -->
-    <!-- base link -->
-    <link name="${prefix}base_link">
-      <inertial>
-        <origin xyz="0 0 0" rpy="0 0 0"/>
-        <mass value="2"/>
-        <inertia ixx="0.01" ixy="0" ixz="0" iyy="0.01" iyz="0" izz="0.01" />
-      </inertial>
-      <visual>
-        <origin xyz="0 0 0" rpy="0 0 0"/>
-        <geometry>
-          <mesh filename="package://kuka_kr16_support/meshes/kr16r2010_2/visual/base_link.stl" />
-        </geometry>
-        <xacro:material_kuka_black />
-      </visual>
-      <collision>
-        <origin xyz="0 0 0" rpy="0 0 0"/>
-        <geometry>
-          <mesh filename="package://kuka_kr16_support/meshes/kr16r2010_2/collision/base_link.stl" />
-        </geometry>
-      </collision>
-    </link>
-    <!-- link 1 (A1) -->
-    <link name="${prefix}link_1">
-      <inertial>
-        <origin xyz="0 0 0" rpy="0 0 0"/>
-        <mass value="2"/>
-        <inertia ixx="0.01" ixy="0" ixz="0" iyy="0.01" iyz="0" izz="0.01" />
-      </inertial>
-      <visual>
-        <origin xyz="0 0 0" rpy="0 0 0"/>
-        <geometry>
-          <mesh filename="package://kuka_kr16_support/meshes/kr16r2010_2/visual/link_1.stl" />
-        </geometry>
-        <xacro:material_kuka_orange />
-      </visual>
-      <collision>
-        <origin xyz="0 0 0" rpy="0 0 0"/>
-        <geometry>
-          <mesh filename="package://kuka_kr16_support/meshes/kr16r2010_2/collision/link_1.stl" />
-        </geometry>
-      </collision>
-    </link>
-    <!-- link 2 -->
-    <link name="${prefix}link_2">
-      <inertial>
-        <origin xyz="0 0 0" rpy="0 0 0"/>
-        <mass value="2"/>
-        <inertia ixx="0.01" ixy="0" ixz="0" iyy="0.01" iyz="0" izz="0.01" />
-      </inertial>
-      <visual>
-        <origin xyz="0 0 0" rpy="0 0 0"/>
-        <geometry>
-          <mesh filename="package://kuka_kr16_support/meshes/kr16r2010_2/visual/link_2.stl"/>
-        </geometry>
-        <xacro:material_kuka_orange />
-      </visual>
-      <collision>
-        <origin xyz="0 0 0" rpy="0 0 0"/>
-        <geometry>
-          <mesh filename="package://kuka_kr16_support/meshes/kr16r2010_2/collision/link_2.stl" />
-        </geometry>
-      </collision>
-    </link>
-    <!-- link 3 -->
-    <link name="${prefix}link_3">
-      <inertial>
-        <origin xyz="0 0 0" rpy="0 0 0"/>
-        <mass value="2"/>
-        <inertia ixx="0.01" ixy="0" ixz="0" iyy="0.01" iyz="0" izz="0.01" />
-      </inertial>
-      <visual>
-        <origin xyz="0 0 0" rpy="0 0 0"/>
-        <geometry>
-          <mesh filename="package://kuka_kr16_support/meshes/kr16r2010_2/visual/link_3.stl" />
-        </geometry>
-        <xacro:material_kuka_orange />
-      </visual>
-      <collision>
-        <origin xyz="0 0 0" rpy="0 0 0"/>
-        <geometry>
-          <mesh filename="package://kuka_kr16_support/meshes/kr16r2010_2/collision/link_3.stl" />
-        </geometry>
-      </collision>
-    </link>
-    <!-- link 4 -->
-    <link name="${prefix}link_4">
-      <inertial>
-        <origin xyz="0 0 0" rpy="0 0 0"/>
-        <mass value="2"/>
-        <inertia ixx="0.01" ixy="0" ixz="0" iyy="0.01" iyz="0" izz="0.01" />
-      </inertial>
-      <visual>
-        <origin xyz="0 0 0" rpy="0 0 0"/>
-        <geometry>
-          <mesh filename="package://kuka_kr16_support/meshes/kr16r2010_2/visual/link_4.stl" />
-        </geometry>
-        <xacro:material_kuka_orange />
-      </visual>
-      <collision>
-        <origin xyz="0 0 0" rpy="0 0 0"/>
-        <geometry>
-          <mesh filename="package://kuka_kr16_support/meshes/kr16r2010_2/collision/link_4.stl" />
-        </geometry>
-      </collision>
-    </link>
-    <!-- link 5 -->
-    <link name="${prefix}link_5">
-      <inertial>
-        <origin xyz="0 0 0" rpy="0 0 0"/>
-        <mass value="2"/>
-        <inertia ixx="0.01" ixy="0" ixz="0" iyy="0.01" iyz="0" izz="0.01" />
-      </inertial>
-      <visual>
-        <origin xyz="0 0 0" rpy="0 0 0"/>
-        <geometry>
-          <mesh filename="package://kuka_kr16_support/meshes/kr16r2010_2/visual/link_5.stl" />
-        </geometry>
-        <xacro:material_kuka_orange />
-      </visual>
-      <collision>
-        <origin xyz="0 0 0" rpy="0 0 0"/>
-        <geometry>
-          <mesh filename="package://kuka_kr16_support/meshes/kr16r2010_2/collision/link_5.stl" />
-        </geometry>
-      </collision>
-    </link>
-    <!-- link 6 -->
-    <link name="${prefix}link_6">
-      <inertial>
-        <origin xyz="0 0 0" rpy="0 0 0"/>
-        <mass value="2"/>
-        <inertia ixx="0.01" ixy="0" ixz="0" iyy="0.01" iyz="0" izz="0.01" />
-      </inertial>
-      <visual>
-        <origin xyz="0 0 0" rpy="0 0 0"/>
-        <geometry>
-          <mesh filename="package://kuka_kr16_support/meshes/kr16r2010_2/visual/link_6.stl" />
-        </geometry>
-        <xacro:material_kuka_pedestal />
-      </visual>
-      <collision>
-        <origin xyz="0 0 0" rpy="0 0 0"/>
-        <geometry>
-          <mesh filename="package://kuka_kr16_support/meshes/kr16r2010_2/collision/link_6.stl" />
-        </geometry>
-      </collision>
-    </link>
-    <!-- tool 0 -->
-    <!-- Following REP199, this frame shall be use to attach EEF or other equipment -->
-    <link name="${prefix}flange" />
-    <!-- END LINKS -->
-    <!-- JOINTS -->
-    <!-- joint 1 (A1) -->
-    <joint name="${prefix}joint_a1" type="revolute">
-      <origin xyz="0.02513108361 0.00023848565 0.27446903331" rpy="0 0 0"/>
-      <parent link="${prefix}base_link"/>
-      <child link="${prefix}link_1"/>
-      <axis xyz="0 0 -1"/>
-      <limit effort="0" lower="${radians(-185)}" upper="${radians(185)}" velocity="${radians(200)}"/>
-    </joint>
-    <!-- joint 2 (A2) -->
-    <joint name="${prefix}joint_a2" type="revolute">
-      <origin xyz="0.160 -0.09480000000 0.24553096669" rpy="${radians(90)} ${radians(90)} ${radians(0)}"/>
-      <parent link="${prefix}link_1"/>
-      <child link="${prefix}link_2"/>
-      <axis xyz="0 0 -1"/>
-      <limit effort="0" lower="${radians(-185)}" upper="${radians(65)}" velocity="${radians(175)}"/>
-    </joint>
-    <!-- joint 3 (A3) -->
-    <joint name="${prefix}joint_a3" type="revolute">
-      <origin xyz="0.0 0.980 0.023" rpy="0 0 ${radians(90)}"/>
-      <parent link="${prefix}link_2"/>
-      <child link="${prefix}link_3"/>
-      <axis xyz="0 0 -1"/>
-      <limit effort="0" lower="${radians(-138)}" upper="${radians(175)}" velocity="${radians(190)}"/>
-    </joint>
-    <!-- joint 4 (A4) -->
-    <joint name="${prefix}joint_a4" type="revolute">
-      <origin xyz="0.3 0.15 -0.1151" rpy="${radians(90)} ${radians(180)} ${radians(90)}"/>
-      <parent link="${prefix}link_3"/>
-      <child link="${prefix}link_4"/>
-      <axis xyz="0 0 -1"/>
-      <limit effort="0" lower="${radians(-350)}" upper="${radians(350)}" velocity="${radians(430)}"/>
-    </joint>
-    <!-- joint 5 (A5) -->
-    <joint name="${prefix}joint_a5" type="revolute">
-      <origin xyz="0 0.0923 0.56000000307" rpy="${radians(90)} ${radians(-90)} ${radians(0)}"/>
-      <parent link="${prefix}link_4"/>
-      <child link="${prefix}link_5"/>
-      <axis xyz="0 0 -1"/>
-      <limit effort="0" lower="${radians(-130)}" upper="${radians(130)}" velocity="${radians(430)}"/>
-    </joint>
-    <!-- joint 6 (A6) -->
-    <joint name="${prefix}joint_a6" type="revolute">
-      <origin xyz="0.139 0.0 0.0923" rpy="${radians(90)} ${radians(180)} ${radians(90)}"/>
-      <parent link="${prefix}link_5"/>
-      <child link="${prefix}link_6"/>
-      <axis xyz="0 0 -1"/>
-      <limit effort="0" lower="${radians(-350)}" upper="${radians(350)}" velocity="${radians(630)}"/>
-    </joint>
-    <!-- tool frame - fixed frame -->
-    <joint name="${prefix}joint_a6-flange" type="fixed">
-      <parent link="${prefix}link_6"/>
-      <child link="${prefix}flange"/>
-      <origin xyz="0.0 0 0.014" rpy="0 0 0"/>
-    </joint>
-    <!-- END JOINTS -->
-    <!-- ROS base_link to KUKA $ROBROOT coordinate system transform -->
-    <link name="${prefix}base" />
-    <joint name="${prefix}base_link-base" type="fixed">
-      <origin xyz="0 0 0" rpy="0 0 0"/>
-      <parent link="${prefix}base_link"/>
-      <child link="${prefix}base"/>
-    </joint>
-    <!-- This frame corresponds to the $TOOL coordinate system in KUKA KRC controllers -->
-    <link name="${prefix}tool0" />
-    <joint name="${prefix}flange-tool0" type="fixed">
-      <parent link="${prefix}flange"/>
-      <child link="${prefix}tool0"/>
-      <origin xyz="0 0 0" rpy="0 ${radians(90)} 0"/>
-    </joint>
-  </xacro:macro>
-</robot>
+<?xml version='1.0' encoding='utf-8'?>
+<robot xmlns:xacro="http://www.ros.org/wiki/xacro">
+    <VERSION value="1.0.0" />
+    <xacro:arg default="" name="prefix" />
+    <xacro:macro name="kuka_kr16r2010_2" params="prefix">
+      <xacro:include filename="$(find kuka_kr16_support)/urdf/kr16r2010_2_params.xacro" />
+      <!--Default materials-->
+      <material name="orange">
+        <color rgba="${246/255} ${120/255} ${40/255} 1" />
+      </material>
+      <material name="black">
+        <color rgba="0 0 0 1" />
+      </material>
+      <!--ROS base_link to KUKA $ROBROOT coordinate system transform-->
+      <link name="${prefix}base" />
+      <!--This frame corresponds to the $TOOL coordinate system in KUKA KRC controllers-->
+      <link name="${prefix}flange" />
+      <joint name="${prefix}joint_flange" type="fixed">
+        <origin rpy="0 0 0" xyz="0 0 0" />
+        <parent link="${prefix}link_6" />
+        <child link="${prefix}flange" />
+      </joint>
+      <link name="${prefix}tool0" />
+      <joint name="${prefix}joint_tool0" type="fixed">
+        <origin rpy="0 0 0" xyz="0 0 0" />
+        <parent link="${prefix}flange" />
+        <child link="${prefix}tool0" />
+      </joint>
+      <!--KR16R2010_2 link-->
+      <link name="${prefix}base_link">
+        <visual>
+          <origin rpy="0 0 0" xyz="0 0 0" />
+          <geometry>
+            <!-- <mesh filename="package://${urdf_package_name}/urdf/robots/kr16r2010_2/meshes/visual/base_link.dae" /> -->
+            <mesh filename="package://kuka_kr16_support/meshes/kr16r2010_2/visual/base_link.dae" />
+          </geometry>
+          <material name="orange" />
+        </visual>
+        <collision>
+          <origin rpy="0 0 0" xyz="0 0 0" />
+          <geometry>
+            <!-- <mesh filename="package://${urdf_package_name}/urdf/robots/kr16r2010_2/meshes/collision/base_link.stl" /> -->
+            <mesh filename="package://kuka_kr16_support/meshes/kr16r2010_2/collision/base_link.stl" />
+          </geometry>
+          <material name="orange" />
+        </collision>
+      </link>
+      <!--KR16R2010_2 joint-->
+      <joint name="${prefix}joint_base_link-base" type="fixed">
+        <origin rpy="${base_link_orientation_r} ${base_link_orientation_p} ${base_link_orientation_y}" xyz="${base_link_origin_x} ${base_link_origin_y} ${base_link_origin_z}" />
+        <parent link="${prefix}base" />
+        <child link="${prefix}base_link" />
+      </joint>
+      <!--A1 link-->
+      <link name="${prefix}link_1">
+        <inertial>
+          <origin rpy="0 0 0" xyz="${link_1_cm_x} ${link_1_cm_y} ${link_1_cm_z}" />
+          <mass value="${link_1_mass}" />
+          <inertia ixx="${link_1_ixx}" ixy="0" ixz="0" iyy="${link_1_iyy}" iyz="0" izz="${link_1_izz}" />
+        </inertial>
+        <visual>
+          <origin rpy="0 0 0" xyz="0 0 0" />
+          <geometry>
+            <!-- <mesh filename="package://${urdf_package_name}/urdf/robots/kr16r2010_2/meshes/visual/link_1.dae" /> -->
+            <mesh filename="package://kuka_kr16_support/meshes/kr16r2010_2/visual/link_1.dae" />
+          </geometry>
+          <material name="orange" />
+        </visual>
+        <collision>
+          <origin rpy="0 0 0" xyz="0 0 0" />
+          <geometry>
+            <!-- <mesh filename="package://${urdf_package_name}/urdf/robots/kr16r2010_2/meshes/collision/link_1.stl" /> -->
+            <mesh filename="package://kuka_kr16_support/meshes/kr16r2010_2/collision/link_1.stl" />
+          </geometry>
+          <material name="orange" />
+        </collision>
+      </link>
+      <!--A1 joint-->
+      <joint name="${prefix}joint_a1" type="revolute">
+        <limit effort="${joint_1_trq}" lower="${radians(joint_1_lower_lim)}" upper="${radians(joint_1_upper_lim)}" velocity="${radians(joint_1_spd)}" />
+        <axis xyz="0 0 -1" />
+        <origin rpy="${link_1_orientation_r} ${link_1_orientation_p} ${link_1_orientation_y}" xyz="${link_1_origin_x} ${link_1_origin_y} ${link_1_origin_z}" />
+        <parent link="${prefix}base_link" />
+        <child link="${prefix}link_1" />
+      </joint>
+      <!--A2 link-->
+      <link name="${prefix}link_2">
+        <inertial>
+          <origin rpy="0 0 0" xyz="${link_2_cm_x} ${link_2_cm_y} ${link_2_cm_z}" />
+          <mass value="${link_2_mass}" />
+          <inertia ixx="${link_2_ixx}" ixy="0" ixz="0" iyy="${link_2_iyy}" iyz="0" izz="${link_2_izz}" />
+        </inertial>
+        <visual>
+          <origin rpy="0 0 0" xyz="0 0 0" />
+          <geometry>
+            <!-- <mesh filename="package://${urdf_package_name}/urdf/robots/kr16r2010_2/meshes/visual/link_2.dae" /> -->
+            <mesh filename="package://kuka_kr16_support/meshes/kr16r2010_2/visual/link_2.dae" />
+          </geometry>
+          <material name="orange" />
+        </visual>
+        <collision>
+          <origin rpy="0 0 0" xyz="0 0 0" />
+          <geometry>
+            <!-- <mesh filename="package://${urdf_package_name}/urdf/robots/kr16r2010_2/meshes/collision/link_2.stl" /> -->
+            <mesh filename="package://kuka_kr16_support/meshes/kr16r2010_2/collision/link_2.stl" />
+          </geometry>
+          <material name="orange" />
+        </collision>
+      </link>
+      <!--A2 joint-->
+      <joint name="${prefix}joint_a2" type="revolute">
+        <limit effort="${joint_2_trq}" lower="${radians(joint_2_lower_lim)}" upper="${radians(joint_2_upper_lim)}" velocity="${radians(joint_2_spd)}" />
+        <axis xyz="0 1 0" />
+        <origin rpy="${link_2_orientation_r} ${link_2_orientation_p} ${link_2_orientation_y}" xyz="${link_2_origin_x} ${link_2_origin_y} ${link_2_origin_z}" />
+        <parent link="${prefix}link_1" />
+        <child link="${prefix}link_2" />
+      </joint>
+      <!--A3 link-->
+      <link name="${prefix}link_3">
+        <inertial>
+          <origin rpy="0 0 0" xyz="${link_3_cm_x} ${link_3_cm_y} ${link_3_cm_z}" />
+          <mass value="${link_3_mass}" />
+          <inertia ixx="${link_3_ixx}" ixy="0" ixz="0" iyy="${link_3_iyy}" iyz="0" izz="${link_3_izz}" />
+        </inertial>
+        <visual>
+          <origin rpy="0 0 0" xyz="0 0 0" />
+          <geometry>
+            <!-- <mesh filename="package://${urdf_package_name}/urdf/robots/kr16r2010_2/meshes/visual/link_3.dae" /> -->
+            <mesh filename="package://kuka_kr16_support/meshes/kr16r2010_2/visual/link_3.dae" />
+          </geometry>
+          <material name="orange" />
+        </visual>
+        <collision>
+          <origin rpy="0 0 0" xyz="0 0 0" />
+          <geometry>
+            <!-- <mesh filename="package://${urdf_package_name}/urdf/robots/kr16r2010_2/meshes/collision/link_3.stl" /> -->
+             <mesh filename="package://kuka_kr16_support/meshes/kr16r2010_2/collision/link_3.stl" />
+          </geometry>
+          <material name="orange" />
+        </collision>
+      </link>
+      <!--A3 joint-->
+      <joint name="${prefix}joint_a3" type="revolute">
+        <limit effort="${joint_3_trq}" lower="${radians(joint_3_lower_lim)}" upper="${radians(joint_3_upper_lim)}" velocity="${radians(joint_3_spd)}" />
+        <axis xyz="0 1 0" />
+        <origin rpy="${link_3_orientation_r} ${link_3_orientation_p} ${link_3_orientation_y}" xyz="${link_3_origin_x} ${link_3_origin_y} ${link_3_origin_z}" />
+        <parent link="${prefix}link_2" />
+        <child link="${prefix}link_3" />
+      </joint>
+      <!--A4 link-->
+      <link name="${prefix}link_4">
+        <inertial>
+          <origin rpy="0 0 0" xyz="${link_4_cm_x} ${link_4_cm_y} ${link_4_cm_z}" />
+          <mass value="${link_4_mass}" />
+          <inertia ixx="${link_4_ixx}" ixy="0" ixz="0" iyy="${link_4_iyy}" iyz="0" izz="${link_4_izz}" />
+        </inertial>
+        <visual>
+          <origin rpy="0 0 0" xyz="0 0 0" />
+          <geometry>
+            <!-- <mesh filename="package://${urdf_package_name}/urdf/robots/kr16r2010_2/meshes/visual/link_4.dae" /> -->
+            <mesh filename="package://kuka_kr16_support/meshes/kr16r2010_2/visual/link_4.dae" />
+          </geometry>
+          <material name="orange" />
+        </visual>
+        <collision>
+          <origin rpy="0 0 0" xyz="0 0 0" />
+          <geometry>
+            <!-- <mesh filename="package://${urdf_package_name}/urdf/robots/kr16r2010_2/meshes/collision/link_4.stl" /> -->
+             <mesh filename="package://kuka_kr16_support/meshes/kr16r2010_2/collision/link_4.stl" />
+          </geometry>
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