Commit message: Add isContinuous parameter for A6 joint type

File: kuka_kr16_support/urdf/kr16r2010_2_macro.xacro (robot description, xacro)
@@ -3,5 +3,6 @@
     <VERSION value="1.0.0" />
     <xacro:arg default="" name="prefix" />
-    <xacro:macro name="kuka_kr16r2010_2" params="prefix">
+    <xacro:property name="isContinuous" value="false"/>
+    <xacro:macro name="kuka_kr16r2010_2" params="prefix isContinuous">
       <xacro:include filename="$(find kuka_kr16_support)/urdf/kr16r2010_2_params.xacro" />
       <!--Default materials-->
@@ -237,5 +238,5 @@
       </link>
       <!--A6 joint-->
-      <joint name="${prefix}joint_a6" type="revolute">
+      <!-- <joint name="${prefix}joint_a6" type="revolute">
         <limit effort="${joint_6_trq}" lower="${radians(joint_6_lower_lim)}" upper="${radians(joint_6_upper_lim)}" velocity="${radians(joint_6_spd)}" />
         <axis xyz="0 0 -1" />
@@ -243,5 +244,22 @@
         <parent link="${prefix}link_5" />
         <child link="${prefix}link_6" />
-      </joint>
+      </joint> -->
+      <xacro:if value="${isContinuous == 'true'}">
+        <joint name="${prefix}joint_a6" type="continuous">
+          <axis xyz="0 0 -1"/>
+          <origin rpy="${link_6_orientation_r} ${link_6_orientation_p} ${link_6_orientation_y}" xyz="${link_6_origin_x} ${link_6_origin_y} ${link_6_origin_z}" />
+          <parent link="${prefix}link_5"/>
+          <child link="${prefix}link_6"/>
+        </joint>
+      </xacro:if>
+      <xacro:unless value="${isContinuous == 'true'}">
+        <joint name="${prefix}joint_a6" type="revolute">
+          <limit effort="${joint_6_trq}" lower="${radians(joint_6_lower_lim)}" upper="${radians(joint_6_upper_lim)}" velocity="${radians(joint_6_spd)}" />
+          <axis xyz="0 0 -1" />
+          <origin rpy="${link_6_orientation_r} ${link_6_orientation_p} ${link_6_orientation_y}" xyz="${link_6_origin_x} ${link_6_origin_y} ${link_6_origin_z}" />
+          <parent link="${prefix}link_5" />
+          <child link="${prefix}link_6" />
+        </joint>
+      </xacro:unless>
     </xacro:macro>
   </robot>
