Commit message: Add necessary KUKA frames

File: kuka_kr300_support/urdf/kr300r2700_2_macro.xacro (robot description, xacro)
@@ -4,4 +4,9 @@
   <xacro:include filename="$(find kuka_resources)/urdf/common_materials.xacro"/>
   <xacro:macro name="kuka_kr300r2700_2" params="prefix">
+      <!--ROS base_link to KUKA $ROBROOT coordinate system transform-->
+    <link name="${prefix}base" />
+    <!--This frame corresponds to the $TOOL coordinate system in KUKA KRC controllers-->
+    <link name="${prefix}flange" />
+    <link name="${prefix}tool0" />
     <!-- links -->
     <link name="${prefix}base_link">
@@ -110,9 +115,10 @@
       </collision>
     </link>
-    <!-- This frame corresponds to the $FLANGE coordinate system in KUKA KRC controllers -->
-    <link name="${prefix}tool0"/>
-    <!-- Following REP199, this frame shall be use to attach EEF or other equipment -->
-    <!-- Add flange ROS-Industrial standard flange -->
-    <link name="${prefix}flange" />
+    <!--KR16R2010_2 joint-->
+    <joint name="${prefix}joint_base_link-base" type="fixed">
+      <origin rpy="0 0 0" xyz="0 0 0" />
+      <parent link="${prefix}base" />
+      <child link="${prefix}base_link" />
+    </joint>
     <!-- Joints -->
     <joint name="${prefix}joint_a1" type="revolute">

Commit message: Remove unnecessary frame and fix tool0 transform

File: kuka_kr300_support/urdf/kr300r2700_2_macro.xacro (robot description, xacro)
@@ -5,5 +5,5 @@
   <xacro:macro name="kuka_kr300r2700_2" params="prefix">
       <!--ROS base_link to KUKA $ROBROOT coordinate system transform-->
-    <link name="${prefix}base" />
+    <!-- <link name="${prefix}base" /> -->
     <!--This frame corresponds to the $TOOL coordinate system in KUKA KRC controllers-->
     <link name="${prefix}flange" />
@@ -116,9 +116,9 @@
     </link>
     <!--KR16R2010_2 joint-->
-    <joint name="${prefix}joint_base_link-base" type="fixed">
+    <!-- <joint name="${prefix}joint_base_link-base" type="fixed">
       <origin rpy="0 0 0" xyz="0 0 0" />
       <parent link="${prefix}base" />
       <child link="${prefix}base_link" />
-    </joint>
+    </joint> -->
     <!-- Joints -->
     <joint name="${prefix}joint_a1" type="revolute">
@@ -158,5 +158,5 @@
     </joint>
     <joint name="${prefix}joint_a6" type="revolute">
-      <origin xyz="0 0 0.2001" rpy="${radians(90)} ${radians(-90)} 0"/>
+      <origin xyz="0 0 0.2001" rpy="${radians(0)} ${radians(-90)} 0"/>
       <parent link="${prefix}link_5"/>
       <child link="${prefix}link_6"/>
@@ -164,11 +164,11 @@
       <limit effort="0" lower="${radians(-350)}" upper="${radians(350)}" velocity="${radians(492)}"/>
     </joint>
-    <joint name="{prefix}link_6-tool0" type="fixed">
-      <origin xyz="0.023 0 0" rpy="0 1.57079632679 0"/>
+    <joint name="${prefix}link_6-tool0" type="fixed">
+      <origin xyz="0.0399 0 0" rpy="0 ${radians(90)} 0"/>
       <parent link="${prefix}link_6"/>
       <child link="${prefix}tool0"/>
     </joint>
     <joint name="${prefix}link_6-flange" type="fixed">
-      <origin xyz="0.023 0 0" rpy="0 1.57079632679 0"/>
+      <origin xyz="0.0399 0 0" rpy="0 ${radians(90)} 0"/>
       <parent link="${prefix}link_6"/>
       <child link="${prefix}flange"/>

Commit message: Fix typo

File: kuka_kr300_support/urdf/kr300r2700_2_macro.xacro (robot description, xacro)
@@ -161,5 +161,5 @@
       <parent link="${prefix}link_5"/>
       <child link="${prefix}link_6"/>
-      <axis xyz="-11 0 0"/>
+      <axis xyz="-1 0 0"/>
       <limit effort="0" lower="${radians(-350)}" upper="${radians(350)}" velocity="${radians(492)}"/>
     </joint>
